File: FC_ESC_STM32F405RG_26x26.kicad_sch (KiCad schematic)
At the start: 194 parts, among them J1 Conn_02x03_Odd_Even, J2 USB_A, Q1 SIZ200, Q10 SIZ200, Q11 SIZ200, Q12 SIZ200, Q2 SIZ200, Q3 SIZ200, Q4 SIZ200, Q5 SIZ200, Q6 SIZ200, Q7 SIZ200, Q8 SIZ200, Q9 SIZ200, SW1 RST, U1 TPS62822DLC, U10 EFM8BB21, U11 FD6288Q, U12 BMP280, U13 ICM-20602, U2 TPS54560BDDA, U3 EFM8BB21, U4 FD6288Q, U5 STM32F405RGTx, U6 EFM8BB21, U7 FD6288Q, U8 EFM8BB21, U9 FD6288Q, Y1 8MHz

Commit message: update project
Parts:
- removed U13: ICM-20602, Package_LGA:LGA-16_3x3mm_P0.5mm_LayoutBorder3x5y, symbol Sensor_Motion:ICM-20602
- added C53: 2.2nF, symbol Device:C_Small
- added C54: 100nF, symbol Device:C_Small
- added D16, D17: SS24, symbol Device:D_Schottky
- added D18: LED_BLUE, symbol Device:LED_Small
- added J10: I2C2_UART3, symbol Connector_Generic:Conn_01x04
- added J11: SD CARD, symbol Connector_Generic:Conn_01x06
- added J12: UART1, symbol Connector_Generic:Conn_01x04
- added J13: UART6, symbol Connector_Generic:Conn_01x04
- added J14: UART4, symbol Connector_Generic:Conn_01x04
- added J15: PWM, symbol Connector_Generic:Conn_01x05
- added J16: UART3, symbol Connector_Generic:Conn_01x04
- added J17: OSD, symbol Connector_Generic:Conn_01x06
- added J18: ALARM, symbol Connector_Generic:Conn_01x02
- added J19: LED_STRIP, symbol Connector_Generic:Conn_01x03
- added J3: Debugger, symbol Connector_Generic:Conn_01x04
- added J4, J5, J6, J7: ESC_PROG, symbol Connector_Generic:Conn_01x03
- added J8: VOL_CUR, symbol Connector_Generic:Conn_01x04
- added J9: RSSI, symbol Connector_Generic:Conn_01x03
- added R79: 10k, symbol Device:R_Small
- added R80, R81: 1k, symbol Device:R_Small
- added R82, R83: 4k7, symbol Device:R_Small
- added R84: 100R, symbol Device:R_Small
- added U13: MPU-6000, symbol EFM8BB21:MPU-6000
- added U14: IP4256CZ5-W, SOT65P210X110-5N, symbol IP4256:IP4256CZ5-W
- C50: value 4.7uF -> 100nF
- C51: value 100nF -> 1nF
- C52: value 2.2uF -> 100nF
- R77: value 4k7 -> 10k
- R78: value 4k7 -> 1k
Connections:
- net +5V: now also J19.1 (Pin_1), J8.1 (Pin_1), J9.1 (Pin_1)
- net 3V3_FC: now also C52.1, D18.2 (A), J10.1 (Pin_1), J11.1 (Pin_1), J12.1 (Pin_1), J13.1 (Pin_1), J14.1 (Pin_1), J16.1 (Pin_1), J17.1 (Pin_1), R79.1, R82.1, R83.1, U13.13 (VDD); no longer C51.1, R78.1, U12.2 (CSB)
- net ESC1_C2CK: now also J4.1 (Pin_1)
- net ESC1_C2D: now also J4.2 (Pin_2)
- net ESC1_RX: now also U5.26 (PB0)
- net ESC2_C2CK: now also J6.1 (Pin_1)
- net ESC2_C2D: now also J6.2 (Pin_2)
- net ESC2_RX: now also U5.27 (PB1)
- net ESC3_C2CK: now also J5.1 (Pin_1)
- net ESC3_C2D: now also J5.2 (Pin_2)
- net ESC3_RX: now also U5.17 (PA3)
- net ESC4_C2CK: now also J7.1 (Pin_1)
- net ESC4_C2D: now also J7.2 (Pin_2)
- net ESC4_RX: now also U5.16 (PA2)
- net GND: now also C53.2, C54.2, J10.4 (Pin_4), J11.6 (Pin_6), J12.4 (Pin_4), J13.4 (Pin_4), J14.4 (Pin_4), J15.5 (Pin_5), J16.4 (Pin_4), J17.6 (Pin_6), J18.2 (Pin_2), J19.3 (Pin_3), J3.4 (Pin_4), J4.3 (Pin_3), J5.3 (Pin_3), J6.3 (Pin_3), J7.3 (Pin_3), J8.4 (Pin_4), J9.3 (Pin_3), U13.1 (CLKIN), U13.11 (FSYNC), U13.18 (GND), U14.2; no longer U12.5 (SDO)
- net STM32_CLK: now also J3.3 (Pin_3)
- net STM32_DIO: now also J3.2 (Pin_2)
- net at C10.1, C9.1, L2.2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: now also D16.2 (A); no longer JP2.1 (A), JP3.1 (A)
- net SENS_VOL: now reaches U5.10 (PC2)
- net SENS_VOL: now also U14.5
- net SENS_RSSI: now reaches U5.14 (PA0)
- net SENS_RSSI: now also J14.2 (Pin_2), R81.2
- net PWM5: now reaches U5.15 (PA1)
- net PWM5: now also J14.3 (Pin_3), J15.1 (Pin_1)
- net IMU_CS: now reaches U5.20 (PA4)
- net IMU_CS: now also R79.2, U13.8 (nCS)
- net IMU_CLK: now reaches U5.21 (PA5)
- net IMU_CLK: now also U13.23 (SCL/SCLK)
- net IMU_MISO: now reaches U5.22 (PA6)
- net IMU_MISO: now also U13.9 (SDO/AD0)
- net IMU_MOSI: now reaches U5.23 (PA7)
- net IMU_MOSI: now also U13.24 (SDA/SD1)
- net IMU_INT: now reaches U5.24 (PC4)
- net IMU_INT: now also U13.12 (INT)
- net STM32_PB10: now reaches U5.29 (PB10)
- net STM32_PB10: now also J10.2 (Pin_2)
- net STM32_PB11: now reaches U5.30 (PB11)
- net STM32_PB11: now also J10.3 (Pin_3)
- net SPI2_CS: now reaches U5.33 (PB12)
- net SPI2_CS: now also J11.2 (Pin_2)
- net SPI2_MOSI: now reaches U5.34 (PB13)
- net SPI2_MOSI: now also J11.3 (Pin_3)
- net SPI2_MISO: now reaches U5.35 (PB14)
- net SPI2_MISO: now also J11.4 (Pin_4)
- net SPI2_CLK: now reaches U5.36 (PB15)
- net SPI2_CLK: now also J11.5 (Pin_5)
- net UART6_TX: now reaches U5.37 (PC6)
- net UART6_TX: now also J13.2 (Pin_2)
- net UART6_RX: now reaches U5.38 (PC7)
- net UART6_RX: now also J13.3 (Pin_3)
- net PWM7: now reaches U5.39 (PC8)
- net PWM7: now also J15.3 (Pin_3)
- net PWM8: now reaches U5.40 (PC9)
- net PWM8: now also J15.4 (Pin_4)
- net PWM6: now reaches U5.41 (PA8)
- net PWM6: now also J15.2 (Pin_2)
- net UART1_TX: now reaches U5.42 (PA9)
- net UART1_TX: now also J12.3 (Pin_3)
- net UART1_RX: now reaches U5.43 (PA10)
- net UART1_RX: now also J12.2 (Pin_2)
- net OSD_CS: now reaches U5.50 (PA15)
- net OSD_CS: now also J17.2 (Pin_2)
- net BARO_CLK: now reaches U5.51 (PC10)
- net BARO_CLK: now also U12.4 (SCK)
- net BARO_MISO: now reaches U5.52 (PC11)
- net BARO_MISO: now also U12.5 (SDO)
- net BARO_MOSI: now reaches U5.53 (PC12)
- net BARO_MOSI: now also U12.3 (SDI)
- net BARO_CS: now reaches U5.55 (PB3)
- net BARO_CS: now also R77.2, U12.2 (CSB)
- net ALARM: now reaches U5.56 (PB4)
- net ALARM: now also J18.1 (Pin_1)
- net LED_BLUE: now reaches U5.57 (PB5)
- net LED_BLUE: now also R84.2
- net LED_STRIP: now reaches U5.58 (PB6)
- net LED_STRIP: now also J19.2 (Pin_2)
- net SENS_CUR: now reaches U5.9 (PC1)
- net SENS_CUR: now also U14.4
- net BMP280_SCK: no longer names the net of R78.2
- net BMP280_SCK: now also U14.1; no longer U12.4 (SCK)
- removed net BMP280_SDI: R77.2, U12.3 (SDI)
- new net: D18.1 (K), R84.1
- new net: C53.1, U13.20 (CPOUT)
- new net: D16.1 (K), D17.1 (K), JP2.1 (A), JP3.1 (A)
- new net: R80.2, U14.3
- new net: C54.1, U13.10 (REGOUT)
- new net 3V3_DEBUGGER: D17.2 (A), J3.1 (Pin_1)
- new net CUR_IN: J8.2 (Pin_2), R80.1
- new net I2C2_SCL: R82.2
- new net I2C2_SDA: R83.2
- new net OSD_CLK: J17.5 (Pin_5)
- new net OSD_MISO: J17.4 (Pin_4)
- new net OSD_MOSI: J17.3 (Pin_3)
- new net RSSI_IN: C51.1, J9.2 (Pin_2), R81.1
- new net UART3_RX: J16.3 (Pin_3)
- new net UART3_TX: J16.2 (Pin_2)
- new net VOL_IN: J8.3 (Pin_3), R78.1
- no-connect marks 22 -> 26
Other:
- note added: "CONNECTOR"
- note added: "VOL-CUR-RSSI"
- moved on the sheet: C24, C25, C26, C52, J1, JP2, JP3, R25, SW1, U12, Y1

Commit message: update current-voltage measure
Parts:
- removed J16: UART3, symbol Connector_Generic:Conn_01x04
- removed J5, J6, J7: ESC_PROG, symbol Connector_Generic:Conn_01x03
- removed U14: IP4256CZ5-W, SOT65P210X110-5N, symbol IP4256:IP4256CZ5-W
- added C55, C56, C57: 100nF, symbol Device:C_Small
- added J20: ESC_PROG, symbol Connector_Generic:Conn_01x09
- added R85, R86: 10k, symbol Device:R_Small
- added R87: Ri_Cur, symbol Device:R_Small
- added R88: Rf_Cur, symbol Device:R_Small
- added R89: Rd_Cur, symbol Device:R_Small
- added U14: LM358, symbol Amplifier_Operational:LM358
- J4: value ESC_PROG -> RC
- R78: value 1k -> Ri_Vol
- R80: value 1k -> Rf_Vol
Connections:
- net +5V: now also J4.1 (Pin_1)
- net 3V3_FC: now also C57.1, U14.8 (V+)
- net 5V_USB: now also R85.1
- net CUR_IN: now also U14.5 (+); no longer R80.1
- net ESC1_C2CK: now also J20.1 (Pin_1); no longer J4.1 (Pin_1)
- net ESC1_C2D: now also J20.2 (Pin_2); no longer J4.2 (Pin_2)
- net ESC2_C2CK: now also J20.3 (Pin_3)
- net ESC2_C2D: now also J20.4 (Pin_4)
- net ESC3_C2CK: now also J20.5 (Pin_5)
- net ESC3_C2D: now also J20.6 (Pin_6)
- net ESC4_C2CK: now also J20.7 (Pin_7)
- net ESC4_C2D: now also J20.8 (Pin_8)
- net GND: now also R78.1, C55.2, C56.2, C57.2, J20.9 (Pin_9), R86.2, R87.1, U14.4 (V-)
- net SENS_CUR: now also C56.1, R89.2
- net SENS_VOL: now also R80.2, C55.1, U14.1
- net SPI2_CLK: now also U5.34 (PB13); no longer U5.36 (PB15)
- net SPI2_MOSI: now also U5.36 (PB15); no longer U5.34 (PB13)
- net VOL_IN: now also U14.3 (+); no longer R78.1
- net at R78.2: now also R80.1, U14.2 (-)
- net SENS_VBUS: now reaches U5.25 (PC5)
- net SENS_VBUS: now also R85.2, R86.1
- net RCIN_INT: now reaches U5.61 (PB8)
- net RCIN_INT: now also J4.2 (Pin_2)
- new net: R88.2, R89.1, U14.7
- new net: R87.2, R88.1, U14.6 (-)
Other:
- moved on the sheet: C51, R81

Commit message: update pcb
Parts:
- removed H1, H10, H11, H12, H2, H3, H4, H5, H6, H7, H8, H9: Motor_Pad, symbol Mechanical:MountingHole_Pad
- removed H13, H14: Battery_Pad, symbol Mechanical:MountingHole_Pad
- removed Q1, Q10, Q11, Q12, Q2, Q3, Q4, Q5, Q6, Q7, Q8, Q9: SIZ200, Package_TO_SOT_THT:TO-220F-5_P3.4x2.06mm_StaggerEven_Lead1.86mm_Vertical, symbol Transistor_FET:IRFI4019H
- added J16, J5, J6, J7: MOTOR, Connector_PinSocket_1.27mm:PinSocket_1x03_P1.27mm_Vertical, symbol Connector_Generic:Conn_01x03
- added J21: ALARM, Connector_PinHeader_2.54mm:PinHeader_1x03_P2.54mm_Vertical, symbol Connector_Generic:Conn_01x03
- added Q1, Q10, Q11, Q13, Q2, Q3, Q4, Q5, Q6, Q7, Q8, Q9: FDS6912, Package_SO:SOIC-8_3.9x4.9mm_P1.27mm, symbol Transistor_FET:FDS6930A
- added U15: outline, Proj_footprint:Board_Outline, symbol Outline:outline
- C1, C10, C11, C2, C27, C29, C31, C36, C38, C43, C45, C6, C7, C8: footprint (none) -> Capacitor_SMD:C_1210_3225Metric
- C12, C13, C14, C15, C16, C17, C18, C19, C20, C21, C22, C23, C24, C25, C26, C28, C3, C30, C32, C33, C34, C35, C37, C39, C4, C40, C41, C42, C44, C46, C47, C48, C49, C5, C50, C51, C52, C53, C54, C55, C56, C57, C9: footprint (none) -> Capacitor_SMD:C_0603_1608Metric
- D1: value 770mV/6A -> S6M_770mV/6A; footprint (none) -> Diode_SMD:D_SMA
- D10, D11, D12, D13, D2, D3, D4, D5, D6, D7, D8, D9: footprint (none) -> Package_TO_SOT_SMD:SOT-23-3
- D14, D15, D16, D17: footprint (none) -> Diode_SMD:D_SMB
- D18: footprint (none) -> LED_SMD:LED_0603_1608Metric
- J1: footprint (none) -> Connector_PinHeader_2.54mm:PinHeader_2x03_P2.54mm_Vertical
- J10, J12, J13, J14, J3, J8: footprint (none) -> Connector_PinHeader_2.54mm:PinHeader_1x04_P2.54mm_Vertical
- J11, J17: footprint (none) -> Connector_PinHeader_2.54mm:PinHeader_1x06_P2.54mm_Vertical
- J15: footprint (none) -> Connector_PinHeader_2.54mm:PinHeader_1x05_P2.54mm_Vertical
- J18: value ALARM -> Conn_01x02; footprint (none) -> Connector_PinHeader_2.54mm:PinHeader_1x02_P2.54mm_Vertical
- J19, J4, J9: footprint (none) -> Connector_PinHeader_2.54mm:PinHeader_1x03_P2.54mm_Vertical
- J2: footprint (none) -> Proj_footprint:USB_Micro-B_2P_4hole
- J20: footprint (none) -> Connector_PinHeader_2.54mm:PinHeader_1x09_P2.54mm_Vertical
- JP1, JP2, JP3, JP4: footprint (none) -> Connector_PinHeader_2.54mm:PinHeader_1x02_P2.54mm_Vertical
- L1: footprint (none) -> Inductor_SMD:L_Bourns_SRP1038C_10.0x10.0mm
- L2: footprint (none) -> Inductor_SMD:L_6.3x6.3_H3
- R1, R10, R11, R12, R13, R14, R15, R16, R17, R18, R19, R2, R20, R21, R22, R23, R24, R25, R26, R27, R28, R29, R3, R30, R31, R32, R33, R34, R35, R36, R37, R38, R39, R4, R40, R41, R42, R43, R44, R45, R46, R47, R48, R49, R5, R50, R51, R52, R53, R54, R55, R56, R57, R58, R59, R6, R60, R61, R62, R63, R64, R65, R66, R67, R68, R69, R7, R70, R71, R72, R73, R74, R75, R76, R77, R78, R79, R8, R80, R81, R82, R83, R84, R85, R86, R87, R88, R89, R9: footprint (none) -> Resistor_SMD:R_0603_1608Metric
- SW1: footprint (none) -> Button_Switch_SMD:SW_Push_SPST_NO_Alps_SKRK
- U10, U3, U6, U8: footprint (none) -> Package_DFN_QFN:SiliconLabs_QFN-20-1EP_3x3mm_P0.5mm_EP1.8x1.8mm
- U11, U4, U7, U9: footprint QFN50P400X400X90-25N -> Package_DFN_QFN:QFN-24-1EP_4x4mm_P0.5mm_EP2.7x2.6mm
- U13: footprint (none) -> Package_DFN_QFN:QFN-24-1EP_4x4mm_P0.5mm_EP2.15x2.15mm
- U14: footprint (none) -> Package_SO:SOIC-8_3.9x4.9mm_P1.27mm
- Y1: footprint (none) -> Crystal:Crystal_SMD_5032-4Pin_5.0x3.2mm
Connections:
- net +5V: now also J21.1 (Pin_1)
- net ALARM: now also J21.2 (Pin_2); no longer J18.1 (Pin_1)
- net ESC1_VS1: now also J5.1 (Pin_1), Q13.3 (S2), Q13.7 (D1), Q13.8 (D1)
- net ESC1_VS2: now also J5.2 (Pin_2), Q1.3 (S2), Q1.7 (D1), Q1.8 (D1)
- net ESC1_VS3: now also J5.3 (Pin_3), Q2.3 (S2), Q2.7 (D1), Q2.8 (D1)
- net ESC2_VS1: now also J6.1 (Pin_1), Q3.3 (S2), Q3.7 (D1), Q3.8 (D1)
- net ESC2_VS2: now also J6.2 (Pin_2), Q4.3 (S2), Q4.7 (D1), Q4.8 (D1)
- net ESC2_VS3: now also J6.3 (Pin_3), Q5.3 (S2), Q5.7 (D1), Q5.8 (D1)
- net ESC3_VS1: now also J7.1 (Pin_1), Q6.3 (S2), Q6.7 (D1), Q6.8 (D1)
- net ESC3_VS2: now also J7.2 (Pin_2), Q7.3 (S2), Q7.7 (D1), Q7.8 (D1)
- net ESC3_VS3: now also J7.3 (Pin_3), Q8.3 (S2), Q8.7 (D1), Q8.8 (D1)
- net ESC4_VS1: now also J16.1 (Pin_1), Q9.3 (S2), Q9.7 (D1), Q9.8 (D1)
- net ESC4_VS2: now also J16.2 (Pin_2), Q10.3 (S2), Q10.7 (D1), Q10.8 (D1)
- net ESC4_VS3: now also J16.3 (Pin_3), Q11.3 (S2), Q11.7 (D1), Q11.8 (D1)
- net GND: now also J21.3 (Pin_3), Q1.1 (S1), Q10.1 (S1), Q11.1 (S1), Q13.1 (S1), Q2.1 (S1), Q3.1 (S1), Q4.1 (S1), Q5.1 (S1), Q6.1 (S1), Q7.1 (S1), Q8.1 (S1), Q9.1 (S1)
- net V_BAT: now also J18.1 (Pin_1), Q1.5 (D2), Q1.6 (D2), Q10.5 (D2), Q10.6 (D2), Q11.5 (D2), Q11.6 (D2), Q13.5 (D2), Q13.6 (D2), Q2.5 (D2), Q2.6 (D2), Q3.5 (D2), Q3.6 (D2), Q4.5 (D2), Q4.6 (D2), Q5.5 (D2), Q5.6 (D2), Q6.5 (D2), Q6.6 (D2), Q7.5 (D2), Q7.6 (D2), Q8.5 (D2), Q8.6 (D2), Q9.5 (D2), Q9.6 (D2)
- net at R62.2: now also Q9.4 (G2)
- net at R39.2: now also Q5.2 (G1)
- net at R51.2: now also Q7.2 (G1)
- net at R50.2: now also Q7.4 (G2)
- net at R15.2: now also Q2.2 (G1)
- net at R14.2: now also Q2.4 (G2)
- net at R46.2: now also Q6.2 (G1)
- net at R45.2: now also Q6.4 (G2)
- net at R56.2: now also Q8.2 (G1)
- net at R12.2: now also Q1.4 (G2)
- net at R73.2: now also Q11.2 (G1)
- net at R72.2: now also Q11.4 (G2)
- net at R63.2: now also Q9.2 (G1)
- net at R28.2: now also Q3.4 (G2)
- net at R29.2: now also Q3.2 (G1)
- net at R68.2: now also Q10.2 (G1)
- net at R55.2: now also Q8.4 (G2)
- net at R34.2: now also Q4.2 (G1)
- net at R33.2: now also Q4.4 (G2)
- net at R11.2: now also Q13.2 (G1)
- net at R10.2: now also Q13.4 (G2)
- net at R38.2: now also Q5.4 (G2)
- net at R67.2: now also Q10.4 (G2)
- net at R13.2: now also Q1.2 (G1)

Commit message: update placement
Parts:
- removed Q1, Q10, Q11, Q13, Q2, Q3, Q4, Q5, Q6, Q7, Q8, Q9: FDS6912, Package_SO:SOIC-8_3.9x4.9mm_P1.27mm, symbol Transistor_FET:FDS6930A
- added Q1, Q10, Q11, Q12, Q2, Q3, Q4, Q5, Q6, Q7, Q8, Q9: SIZ200, Proj_footprint:ONSC-WDFN-8-511AB_V, symbol Transistor_FET:IRFI4019H
- D12: renamed from D3; footprint Package_TO_SOT_SMD:SOT-23-3 -> Diode_SMD:D_SOD-123F
- D13: renamed from D11; footprint Package_TO_SOT_SMD:SOT-23-3 -> Diode_SMD:D_SOD-123F
- D14: renamed from D4; footprint Package_TO_SOT_SMD:SOT-23-3 -> Diode_SMD:D_SOD-123F
- D15: renamed from D12; footprint Package_TO_SOT_SMD:SOT-23-3 -> Diode_SMD:D_SOD-123F
- D16: renamed from D7; footprint Package_TO_SOT_SMD:SOT-23-3 -> Diode_SMD:D_SOD-123F
- D17: renamed from D13; footprint Package_TO_SOT_SMD:SOT-23-3 -> Diode_SMD:D_SOD-123F
- D2: footprint Package_TO_SOT_SMD:SOT-23-3 -> Diode_SMD:D_SOD-123F
- D3: renamed from D8; footprint Package_TO_SOT_SMD:SOT-23-3 -> Diode_SMD:D_SOD-123F
- D6: renamed from D5; footprint Package_TO_SOT_SMD:SOT-23-3 -> Diode_SMD:D_SOD-123F
- D7: renamed from D9; footprint Package_TO_SOT_SMD:SOT-23-3 -> Diode_SMD:D_SOD-123F
- D8: renamed from D6; footprint Package_TO_SOT_SMD:SOT-23-3 -> Diode_SMD:D_SOD-123F
- D9: renamed from D10; footprint Package_TO_SOT_SMD:SOT-23-3 -> Diode_SMD:D_SOD-123F
- L1: footprint Inductor_SMD:L_Bourns_SRP1038C_10.0x10.0mm -> Inductor_SMD:L_Chilisin_BMRA00040420
- Y1: footprint Crystal:Crystal_SMD_5032-4Pin_5.0x3.2mm -> Crystal:Crystal_SMD_3225-4Pin_3.2x2.5mm
- renumbered C11 to C1, C38 to C10, C28 to C11, C39 to C12, C5 to C13, C6 to C14, C7 to C15, C13 to C16, C40 to C17, C16 to C18, C41 to C19, C36 to C2, C8 to C20, C17 to C21, C42 to C22, C29 to C23, C43 to C24, C30 to C25, C44 to C26, C9 to C27, C10 to C28, C31 to C29, C12 to C3, C45 to C30, C32 to C31, C46 to C32, C47 to C34, C34 to C35, C48 to C36, C35 to C37, C49 to C38, C52 to C39, C37 to C4, C50 to C40, C54 to C41, C53 to C42, C26 to C43, C24 to C44, C25 to C45, C23 to C46, C22 to C47, C14 to C48, C15 to C49, C2 to C5, C18 to C50, C19 to C52, C57 to C53, C55 to C54, C56 to C55, C20 to C56, C21 to C57, C1 to C6, C3 to C7, C4 to C8, C27 to C9, D17 to D10, D16 to D11, D14 to D4, D15 to D5, J18 to J1, J14 to J10, J15 to J11, J17 to J12, J21 to J13, J19 to J14, J4 to J15, J7 to J16, J5 to J17, J6 to J18, J16 to J19, J20 to J2, J2 to J20, J1 to J21, J8 to J4, J9 to J5, J10 to J6, J11 to J7, J12 to J8, J13 to J9, JP4 to JP1, JP1 to JP2, JP2 to JP3, JP3 to JP4, R8 to R1, R23 to R10, R47 to R11, R48 to R12, R24 to R13, R49 to R14, R1 to R15, R2 to R16, R12 to R17, R13 to R18, R50 to R19, R43 to R2, R51 to R20, R19 to R21, R20 to R22, R52 to R23, R53 to R24, R21 to R25, R54 to R26, R3 to R27, R4 to R28, R14 to R29, R9 to R3, R15 to R30, R55 to R31, R56 to R32, R18 to R33, R16 to R34, R57 to R35, R58 to R36, R17 to R37, R59 to R38, R5 to R39, R10 to R4, R26 to R40, R60 to R41, R27 to R42, R28 to R43, R29 to R44, R61 to R45, R62 to R46, R63 to R47, R30 to R48, R31 to R49, R11 to R5, R64 to R50, R65 to R51, R6 to R52, R7 to R53, R32 to R54, R66 to R55, R33 to R56, R34 to R57, R67 to R58, R68 to R59, R44 to R6, R35 to R60, R36 to R61, R69 to R62, R70 to R63, R37 to R64, R71 to R65, R38 to R66, R39 to R67, R72 to R68, R73 to R69, R45 to R7, R40 to R70, R41 to R71, R74 to R72, R75 to R73, R42 to R74, R76 to R75, R79 to R76, R85 to R77, R86 to R78, R77 to R79, R46 to R8, R84 to R80, R83 to R81, R25 to R83, R78 to R84, R87 to R85, R80 to R86, R88 to R87, R89 to R88, R81 to R89, R22 to R9, U3 to U1, U11 to U10, U15 to U11, U13 to U12, U12 to U13, U5 to U15, U8 to U2, U2 to U3, U9 to U5, U1 to U6, U6 to U7, U10 to U8, U7 to U9
Connections:
- net ESC1_VS1: now also Q1.3 (S1/D2)
- net ESC1_VS2: now also Q3.3 (S1/D2)
- net ESC1_VS3: now also Q5.3 (S1/D2)
- net ESC2_VS1: now also Q7.3 (S1/D2)
- net ESC2_VS2: now also Q9.3 (S1/D2)
- net ESC2_VS3: now also Q11.3 (S1/D2)
- net ESC3_VS1: now also Q2.3 (S1/D2)
- net ESC3_VS2: now also Q4.3 (S1/D2)
- net ESC3_VS3: now also Q6.3 (S1/D2)
- net ESC4_VS1: now also Q8.3 (S1/D2)
- net ESC4_VS2: now also Q10.3 (S1/D2)
- net ESC4_VS3: now also Q12.3 (S1/D2)
- net GND: now also Q1.1 (S2), Q10.1 (S2), Q11.1 (S2), Q12.1 (S2), Q2.1 (S2), Q3.1 (S2), Q4.1 (S2), Q5.1 (S2), Q6.1 (S2), Q7.1 (S2), Q8.1 (S2), Q9.1 (S2)
- net V_BAT: now also Q1.5 (D1), Q10.5 (D1), Q11.5 (D1), Q12.5 (D1), Q2.5 (D1), Q3.5 (D1), Q4.5 (D1), Q5.5 (D1), Q6.5 (D1), Q7.5 (D1), Q8.5 (D1), Q9.5 (D1)
- net at R31.2: now also Q6.4 (G1)
- net at R46.2: now also Q8.4 (G1)
- net at R67.2: now also Q11.2 (G2)
- net at R29.2: now also Q5.4 (G1)
- net at R66.2: now also Q11.4 (G1)
- net at C44.1, U15.5 (PH0): now also Y1.2; no longer Y1.1
- net at R57.2: now also Q9.2 (G2)
- net at C45.1, U15.6 (PH1): now also Y1.1; no longer Y1.2
- net at R58.2: now also Q10.4 (G1)
- net at R32.2: now also Q6.2 (G2)
- net at R17.2: now also Q3.4 (G1)
- net at R4.2: now also Q1.4 (G1)
- net at R43.2: now also Q7.4 (G1)
- net at R44.2: now also Q7.2 (G2)
- net at R19.2: now also Q4.4 (G1)
- net at R20.2: now also Q4.2 (G2)
- net at R8.2: now also Q2.2 (G2)
- net at R30.2: now also Q5.2 (G2)
- net at R59.2: now also Q10.2 (G2)
- net at R68.2: now also Q12.4 (G1)
- net at R47.2: now also Q8.2 (G2)
- net at R56.2: now also Q9.4 (G1)
- net at R18.2: now also Q3.2 (G2)
- net at R69.2: now also Q12.2 (G2)
- net at R5.2: now also Q1.2 (G2)
- net at R7.2: now also Q2.4 (G1)

Commit message: update placement
Parts:
- C11, C12, C13, C16, C17, C18, C19, C21, C22, C25, C26, C27, C3, C31, C32, C33, C34, C35, C36, C37, C38, C39, C4, C40, C41, C42, C43, C44, C45, C46, C47, C48, C49, C50, C51, C52, C53, C54, C55, C56, C57, C7, C8: footprint Capacitor_SMD:C_0603_1608Metric -> Capacitor_SMD:C_0402_1005Metric_Pad0.74x0.62mm_HandSolder
- J16, J17, J18, J19: footprint Connector_PinSocket_1.27mm:PinSocket_1x03_P1.27mm_Vertical -> Proj_footprint:Hirose_DF13-03P-1.25DS_1x03_P1.25mm_Horizontal
- R1, R10, R11, R12, R13, R14, R15, R16, R17, R18, R19, R2, R20, R21, R22, R23, R24, R25, R26, R27, R28, R29, R3, R30, R31, R32, R33, R34, R35, R36, R37, R38, R39, R4, R40, R41, R42, R43, R44, R45, R46, R47, R48, R49, R5, R50, R51, R52, R53, R54, R55, R56, R57, R58, R59, R6, R60, R61, R62, R63, R64, R65, R66, R67, R68, R69, R7, R70, R71, R72, R73, R74, R75, R76, R77, R78, R79, R8, R80, R81, R82, R83, R84, R85, R86, R87, R88, R89, R9: footprint Resistor_SMD:R_0603_1608Metric -> Resistor_SMD:R_0402_1005Metric_Pad0.72x0.64mm_HandSolder
- U1, U2, U7, U8: footprint Package_DFN_QFN:SiliconLabs_QFN-20-1EP_3x3mm_P0.5mm_EP1.8x1.8mm -> Proj_footprint:QFN-20-1EP_3x3mm_P0.5mm_EP1.8x1.8mm
- U12: footprint Package_DFN_QFN:QFN-24-1EP_4x4mm_P0.5mm_EP2.15x2.15mm -> Proj_footprint:QFN-24-1EP_4x4mm_P0.5mm_EP2.15x2.15mm

Commit message: update placement
Parts:
- removed C11, C12, C25, C26, C3, C31, C32, C4: 100nF, Capacitor_SMD:C_0402_1005Metric_Pad0.74x0.62mm_HandSolder, symbol Device:C_Small
- C1, C2: footprint Capacitor_SMD:C_1210_3225Metric -> Capacitor_SMD:C_0603_1608Metric_Pad1.08x0.95mm_HandSolder
- C10: renamed from C14; footprint Capacitor_SMD:C_1210_3225Metric -> Capacitor_SMD:C_0805_2012Metric_Pad1.18x1.45mm_HandSolder
- C11: renamed from C15; footprint Capacitor_SMD:C_1210_3225Metric -> Capacitor_SMD:C_0805_2012Metric_Pad1.18x1.45mm_HandSolder
- C16: renamed from C20; footprint Capacitor_SMD:C_1210_3225Metric -> Capacitor_SMD:C_0805_2012Metric_Pad1.18x1.45mm_HandSolder
- C19: renamed from C23; footprint Capacitor_SMD:C_1210_3225Metric -> Capacitor_SMD:C_0603_1608Metric_Pad1.08x0.95mm_HandSolder
- C20: renamed from C24; footprint Capacitor_SMD:C_1210_3225Metric -> Capacitor_SMD:C_0603_1608Metric_Pad1.08x0.95mm_HandSolder
- C22: renamed from C28; footprint Capacitor_SMD:C_1210_3225Metric -> Capacitor_SMD:C_0805_2012Metric_Pad1.18x1.45mm_HandSolder
- C23: renamed from C29; value 4.7uF -> 100nF; footprint Capacitor_SMD:C_1210_3225Metric -> Capacitor_SMD:C_0402_1005Metric_Pad0.74x0.62mm_HandSolder
- C24: renamed from C30; value 4.7uF -> 100nF; footprint Capacitor_SMD:C_1210_3225Metric -> Capacitor_SMD:C_0402_1005Metric_Pad0.74x0.62mm_HandSolder
- C3: renamed from C5; footprint Capacitor_SMD:C_1210_3225Metric -> Capacitor_SMD:C_0805_2012Metric_Pad1.18x1.45mm_HandSolder
- C4: renamed from C6; footprint Capacitor_SMD:C_1210_3225Metric -> Capacitor_SMD:C_0805_2012Metric_Pad1.18x1.45mm_HandSolder
- C7: renamed from C9; value 4.7uF -> 100nF; footprint Capacitor_SMD:C_1210_3225Metric -> Capacitor_SMD:C_0402_1005Metric_Pad0.74x0.62mm_HandSolder
- C8: renamed from C10; value 4.7uF -> 100nF; footprint Capacitor_SMD:C_1210_3225Metric -> Capacitor_SMD:C_0402_1005Metric_Pad0.74x0.62mm_HandSolder
- D12, D13, D14, D15, D16, D17, D2, D3, D6, D7, D8, D9: footprint Diode_SMD:D_SOD-123F -> Diode_SMD:D_SOD-323
- renumbered C16 to C12, C17 to C13, C18 to C14, C19 to C15, C21 to C17, C22 to C18, C27 to C21, C33 to C25, C34 to C26, C35 to C27, C36 to C28, C37 to C29, C38 to C30, C39 to C31, C40 to C32, C41 to C33, C42 to C34, C43 to C35, C44 to C36, C45 to C37, C46 to C38, C47 to C39, C48 to C40, C49 to C41, C50 to C42, C51 to C43, C52 to C44, C53 to C45, C54 to C46, C55 to C47, C56 to C48, C57 to C49, C7 to C5, C8 to C6, C13 to C9

Commit message: update placement
Parts:
- removed C2, C20: 4.7uF, Capacitor_SMD:C_0603_1608Metric_Pad1.08x0.95mm_HandSolder, symbol Device:C_Small
- removed J1: Conn_01x02, Connector_PinHeader_2.54mm:PinHeader_1x02_P2.54mm_Vertical, symbol Connector_Generic:Conn_01x02
- added C50, C51, C52, C53: 4.7uF, Capacitor_SMD:C_0603_1608Metric_Pad1.08x0.95mm_HandSolder, symbol Device:C_Small
- added C54, C55, C56, C57: 100nF, Capacitor_SMD:C_0402_1005Metric_Pad0.74x0.62mm_HandSolder, symbol Device:C_Small
- added D19: SS54, Diode_SMD:D_SMB, symbol Device:D_Small
- added H1: VBAT, Proj_footprint:MoutingPad, symbol Mechanical:MountingHole_Pad
- added H2: GND, Proj_footprint:MoutingPad, symbol Mechanical:MountingHole_Pad
- C1, C19: footprint Capacitor_SMD:C_0603_1608Metric_Pad1.08x0.95mm_HandSolder -> Capacitor_SMD:C_1206_3216Metric_Pad1.33x1.80mm_HandSolder
- C10, C11, C3, C4: footprint Capacitor_SMD:C_0805_2012Metric_Pad1.18x1.45mm_HandSolder -> Capacitor_SMD:C_1210_3225Metric_Pad1.33x2.70mm_HandSolder
- U3: footprint Package_SO:Texas_R-PDSO-G8_EP2.95x4.9mm_Mask2.4x3.1mm_ThermalVias -> Proj_footprint:PDSO-G8_EP2.95x4.9mm_Mask2.4x3.1mm
Connections:
- net +5V: now also C50.1, C51.1, C52.1, C53.1
- net 3V3_ESC: now also C54.1, C55.1, C56.1, C57.1
- net GND: now also C50.2, C51.2, C52.2, C53.2, C54.2, C55.2, C56.2, C57.2, D19.2 (A), H2.1
- net V_BAT: now also D19.1 (K), H1.1
Other:
- moved on the sheet: C10, C11, C16, C21, C22, C3, C4, C5, C6, C9, D1, D10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
