File: FC_ESC_STM32F405RG_26x26.kicad_sch (KiCad schematic)
At the start: 220 parts, among them J10 UART4, J11 PWM, J12 OSD, J13 ALARM, J14 LED_STRIP, J15 RC, J16 MOTOR, J17 MOTOR, J18 MOTOR, J19 MOTOR, J2 ESC_PROG, J20 USB_A, J21 Conn_02x03_Odd_Even, J3 Debugger, J4 VOL_CUR, J5 RSSI, J6 I2C2_UART3, J7 SD CARD, J8 UART1, J9 UART6, Q1 SIZ200, Q10 SIZ200, Q11 SIZ200, Q12 SIZ200, Q2 SIZ200, Q3 SIZ200, Q4 SIZ200, Q5 SIZ200, Q6 SIZ200, Q7 SIZ200, Q8 SIZ200, Q9 SIZ200, SW1 RST, U1 EFM8BB21, U10 FD6288Q, U11 outline, U12 MPU-6000, U13 BMP280, U14 LM358, U15 STM32F405RGTx, U2 EFM8BB21, U3 TPS54560BDDA, U4 FD6288Q, U5 FD6288Q, U6 TPS62822DLC, U7 EFM8BB21, U8 EFM8BB21, U9 FD6288Q, Y1 8MHz

Commit message: update placement
Parts:
- removed J20: USB_A, Proj_footprint:USB_Micro-B_2P_4hole, symbol Connector:USB_A
- removed JP1: Jumper_5V, Connector_PinHeader_2.54mm:PinHeader_1x02_P2.54mm_Vertical, symbol Jumper:Jumper_2_Open
- removed JP2: Jumper_5V_PWR, Connector_PinHeader_2.54mm:PinHeader_1x02_P2.54mm_Vertical, symbol Jumper:Jumper_2_Open
- removed R39: 100k, Resistor_SMD:R_0402_1005Metric_Pad0.72x0.64mm_HandSolder, symbol Device:R_Small
- removed U6: TPS62822DLC, Package_DFN_QFN:Texas_VSON-HR-8_1.5x2mm_P0.5mm, symbol Regulator_Switching:TPS62822DLC
- added C2: 1nF, Capacitor_SMD:C_0402_1005Metric_Pad0.74x0.62mm_HandSolder, symbol Device:C_Small
- added C20: 10pF, Capacitor_SMD:C_0402_1005Metric_Pad0.74x0.62mm_HandSolder, symbol Device:C_Small
- added C58: 8.2nF, Capacitor_SMD:C_0402_1005Metric_Pad0.74x0.62mm_HandSolder, symbol Device:C_Small
- added D20: SS34, Diode_SMD:D_SMA, symbol Device:D_Small
- added J1: USB, Connector_Hirose:Hirose_DF3EA-04P-2H_1x04-1MP_P2.00mm_Horizontal, symbol Connector_Generic:Conn_01x04
- added J22: Conn_02x02_Odd_Even, Connector_PinHeader_1.27mm:PinHeader_2x02_P1.27mm_Vertical_SMD, symbol Connector_Generic:Conn_02x02_Odd_Even
- added R90: 28.7k, Resistor_SMD:R_0402_1005Metric_Pad0.72x0.64mm_HandSolder, symbol Device:R_Small
- added U16: TPS54331D, Package_SO:SOIC-8-1EP_3.9x4.9mm_P1.27mm_EP2.29x3mm, symbol TPS54331:TPS54331D
- C21: value 120pF -> 100nF
- D4, D5: value SS24 -> SS34; footprint Diode_SMD:D_SMB -> Diode_SMD:D_SMA
- L1: footprint Inductor_SMD:L_Chilisin_BMRA00040420 -> Proj_footprint:Inductor
- L2: value 470nH -> 4uH; footprint Inductor_SMD:L_6.3x6.3_H3 -> Proj_footprint:Inductor
- R16: value 274k -> 274k
- R52: value 453k -> 10k2
- R53: value 100k -> 3.24k
Connections:
- net +5V: now also J22.2 (Pin_2)
- net 5V_USB: now also J1.1 (Pin_1)
- net GND: now also C2.2, C20.2, C58.2, D20.2 (A), J1.4 (Pin_4), U16.7 (GND)
- net USB_D+: now also J1.2 (Pin_2)
- net USB_D-: now also J1.3 (Pin_3)
- net at D4.1 (K), D5.1 (K): now also J22.1 (Pin_1), J22.3 (Pin_3); no longer C16.1
- net at C22.1, D11.2 (A), L2.2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: no longer C21.1
- net at R52.2, R53.1: now also U16.5 (VSENSE); no longer C21.2
- net at L2.1: now also C21.2, D20.1 (K), U16.8 (PH)
- new net: C16.1, J22.4 (Pin_4), U16.2 (VIN)
- new net: C58.1, U16.4 (SS)
- new net: C21.1, U16.1 (BOOT)
- new net: C20.1, R90.2, U16.6 (COMP)
- new net: C2.1, R90.1
- no-connect marks 26 -> 27
Other:
- note added: "Imax 3A"
- note removed: "Imax 1.5A"
- moved on the sheet: C16, C21, C22, D10, D11, JP3, JP4, L2, R52, R53, U11
