File: FC_ESC_STM32F405RG_26x26.kicad_sch (KiCad schematic)
At the start: 223 parts, among them J1 Conn_01x02, J10 Conn_01x01, J11 Conn_01x02, J12 Conn_02x02_Odd_Even, J13 ALARM, J14 LED_STRIP, J16 MOTOR, J17 MOTOR, J18 MOTOR, J19 MOTOR, J2 Conn_02x04_Odd_Even, J20 USB_A, J21 ESC_PROG, J23 ESC_PROG, J24 ESC_PROG, J25 ESC_PROG, J3 Debugger, J4 Conn_01x04, J5 RSSI, J6 Conn_01x04, J7 Conn_01x02, J8 Conn_01x04, J9 LED_STRIP, Q1 SIZ200, Q10 SIZ200, Q11 SIZ200, Q12 SIZ200, Q2 SIZ200, Q3 SIZ200, Q4 SIZ200, Q5 SIZ200, Q6 SIZ200, Q7 SIZ200, Q8 SIZ200, Q9 SIZ200, U1 EFM8BB21, U10 FD6288Q, U11 outline, U12 MPU-6000, U13 BMP280, U15 STM32F405RGTx, U16 RT9013-33GB, U2 EFM8BB21, U3 TPS54560BDDA, U4 FD6288Q, U5 FD6288Q, U6 AT7456, U7 EFM8BB21, U8 EFM8BB21, U9 FD6288Q, Y1 8MHz, Y2 8Mhz

Commit message: update placement
Parts:
- removed D19: SS34, Diode_SMD:D_SMA, symbol Device:D_Small
- removed J10: Conn_01x01, Proj_footprint:MountingPad_1x1, symbol Connector_Generic:Conn_01x01
- removed J11: Conn_01x02, Proj_footprint:MountingPad_1x2, symbol Connector_Generic:Conn_01x02
- removed J13: ALARM, Proj_footprint:MountingPad_1x3, symbol Connector_Generic:Conn_01x03
- removed J14, J9: LED_STRIP, Proj_footprint:MountingPad_1x3, symbol Connector_Generic:Conn_01x03
- removed J5: RSSI, Proj_footprint:MountingPad_1x3, symbol Connector_Generic:Conn_01x03
- removed J6: Conn_01x04, Proj_footprint:MountingPad_1x4, symbol Connector_Generic:Conn_01x04
- removed J7: Conn_01x02, Proj_footprint:MountingPad_5VOUT, symbol Connector_Generic:Conn_01x02
- added J10: LED_STRIP, Proj_footprint:MountingPad_1x3, symbol Connector_Generic:Conn_01x03
- added J14, J15, J26, J5, J9: Conn_01x04, Proj_footprint:MountingPad_1x4, symbol Connector_Generic:Conn_01x04
- added J6: Conn_01x02, Proj_footprint:MountingPad_1x2, symbol Connector_Generic:Conn_01x02
- C2: footprint Capacitor_SMD:C_1210_3225Metric_Pad1.33x2.70mm_HandSolder -> Capacitor_SMD:C_1206_3216Metric_Pad1.33x1.80mm_HandSolder
- D18, D4, D5: footprint LED_SMD:LED_0603_1608Metric -> LED_SMD:LED_0402_1005Metric_Pad0.77x0.64mm_HandSolder
- J1: footprint Proj_footprint:MountingPad_5VOUT -> Proj_footprint:MountingPad_1x2
- J20: footprint Proj_footprint:USB_Micro-B_2P_4hole -> Proj_footprint:USB_Micro-B_SMD
Connections:
- net +5V: now also J1.1 (Pin_1), J4.1 (Pin_1), J8.1 (Pin_1), J10.1 (Pin_1), J14.1 (Pin_1), J15.1 (Pin_1), J26.1 (Pin_1), J6.1 (Pin_1), J9.1 (Pin_1); no longer J1.2 (Pin_2)
- net ALARM: now also J26.3 (Pin_3)
- net GND: now also J1.2 (Pin_2), J4.4 (Pin_4), J8.4 (Pin_4), J10.3 (Pin_3), J14.4 (Pin_4), J15.4 (Pin_4), J26.4 (Pin_4), J6.2 (Pin_2), J9.4 (Pin_4); no longer J1.1 (Pin_1)
- net LED_STRIP: now also J26.2 (Pin_2)
- net OSD_VIDEO_IN: now also J9.3 (Pin_3)
- net OSD_VIDEO_OUT: now also J9.2 (Pin_2)
- net RCIN_INT: now also J10.2 (Pin_2)
- net SENS_RSSI: now also J4.2 (Pin_2); no longer J4.1 (Pin_1)
- net SPI2_CLK: now also J5.4 (Pin_4)
- net SPI2_CS: now also J5.1 (Pin_1)
- net SPI2_MISO: now also J5.3 (Pin_3)
- net SPI2_MOSI: now also J5.2 (Pin_2)
- net STM32_PA1: now also J4.3 (Pin_3); no longer J4.2 (Pin_2)
- net STM32_PB10: now also J15.2 (Pin_2); no longer J4.3 (Pin_3)
- net STM32_PB11: now also J15.3 (Pin_3); no longer J4.4 (Pin_4)
- net UART1_RX: now also J14.2 (Pin_2); no longer J8.3 (Pin_3)
- net UART1_TX: now also J14.3 (Pin_3); no longer J8.4 (Pin_4)
- net UART6_RX: now also J8.3 (Pin_3); no longer J8.2 (Pin_2)
- net UART6_TX: now also J8.2 (Pin_2); no longer J8.1 (Pin_1)
- net PWM_OUT: no longer names the net of U15.39 (PC8)
Other:
- moved on the sheet: J4, J8

Commit message: update placement
Parts:
- removed C22: 100uF, Capacitor_SMD:C_1206_3216Metric_Pad1.33x1.80mm_HandSolder, symbol Device:C_Small
- removed C65: 100nF, Capacitor_SMD:C_0402_1005Metric_Pad0.74x0.62mm_HandSolder, symbol Device:C_Small
- removed D4: LED_RED, LED_SMD:LED_0402_1005Metric_Pad0.77x0.64mm_HandSolder, symbol Device:LED_Small
- removed J1, J6: Conn_01x02, Proj_footprint:MountingPad_1x2, symbol Connector_Generic:Conn_01x02
- removed J10: LED_STRIP, Proj_footprint:MountingPad_1x3, symbol Connector_Generic:Conn_01x03
- removed J5: Conn_01x04, Proj_footprint:MountingPad_1x4, symbol Connector_Generic:Conn_01x04
- removed R41: 1k, Resistor_SMD:R_0402_1005Metric_Pad0.72x0.64mm_HandSolder, symbol Device:R_Small
- removed R92: 100R, Resistor_SMD:R_0402_1005Metric_Pad0.72x0.64mm_HandSolder, symbol Device:R_Small
- added J1: Conn_01x06, Proj_footprint:MountingPad_1x6, symbol Connector_Generic:Conn_01x06
- added J7: Conn_01x04, Proj_footprint:MountingPad_1x4, symbol Connector_Generic:Conn_01x04
- C2: footprint Capacitor_SMD:C_1206_3216Metric_Pad1.33x1.80mm_HandSolder -> Capacitor_SMD:C_1210_3225Metric_Pad1.33x2.70mm_HandSolder
- C50, C51, C52, C53: footprint Capacitor_SMD:C_0603_1608Metric_Pad1.08x0.95mm_HandSolder -> Capacitor_SMD:C_0402_1005Metric_Pad0.74x0.62mm_HandSolder
- R1, R2, R40: value 1k -> 2k2
Connections:
- net +5V: now also J1.1 (Pin_1), J7.1 (Pin_1)
- net 3V3_FC: now also R1.1, R40.1; no longer R87.2, U15.60 (BOOT0)
- net ESC1_RX: now also U1.2 (P0.0); no longer R1.1
- net ESC2_RX: now also U7.2 (P0.0); no longer R40.1
- net ESC3_RX: now also U2.2 (P0.0); no longer R2.1
- net ESC4_RX: now also U8.2 (P0.0)
- net GND: now also R2.1, J1.6 (Pin_6), J7.4 (Pin_4)
- net LED_PWR_3V3: now also C2.1
- net RCIN_INT: now also J7.2 (Pin_2)
- net RSSI_IN: now also J7.3 (Pin_3)
- net SPI2_CLK: now also J1.5 (Pin_5)
- net SPI2_CS: now also J1.2 (Pin_2)
- net SPI2_MISO: now also J1.4 (Pin_4)
- net SPI2_MOSI: now also J1.3 (Pin_3)
- net at Y2.1: now also U6.6 (XFB); no longer U6.5 (CLKIN)
- net at Y2.2: now also U6.5 (CLKIN); no longer U6.6 (XFB)
- net at J2.3 (Pin_3), U16.5 (VOUT): no longer C2.1
- net BOOT0: now reaches R1.2
- net BOOT0: now also R87.2, U15.60 (BOOT0); no longer U1.2 (P0.0)
- net BOOT1: now reaches R40.2
- net BOOT1: now also R2.2, U15.28 (PB2); no longer U7.2 (P0.0)
- net LED_PWR_5V: no longer names the net of C10.1, C16.1, J12.3 (Pin_3), L1.2, R27.1
Other:
- moved on the sheet: C2, R87

Commit message: update schematic
Parts:
- J1: value Conn_01x06 -> SPI
- J14: value Conn_01x04 -> UART1
- J15: value Conn_01x04 -> UART3_I2C2
- J26: value Conn_01x04 -> LED_BUZ
- J3: value Debugger -> ST-LINK
- J4: value Conn_01x04 -> UART4
- J7: value Conn_01x04 -> RC
- J8: value Conn_01x04 -> UART6
- J9: value Conn_01x04 -> OSD
- U11: value outline -> OUTLINE
Other:
- note added: "BMP280"
- note added: "ESC PROG"
- note added: "MOTOR"
- note added: "MPU6000"
- note added: "OUTLINE"
- note added: "POWER"
- note added: "RESOURCE"
- note added: "STM32F405RG"
- note added: "USB"
- note removed: "BAROMETER"
- note removed: "IMU"
- note removed: "Imax 3A"
- note removed: "POWER SUPPLY"
- note removed: "STM32F4"
- moved on the sheet: C10, C16, C2, C3, C36, C37, C38, C39, C4, C40, C41, C42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

Commit message: update routing
Parts:
- removed Q1, Q10, Q11, Q12, Q2, Q3, Q4, Q5, Q6, Q7, Q8, Q9: SIZ200, Proj_footprint:ONSC-WDFN-8-511AB_V, symbol Transistor_FET:IRFI4019H
- removed R1, R2, R40: 2k2, Resistor_SMD:R_0402_1005Metric_Pad0.72x0.64mm_HandSolder, symbol Device:R_Small
- added U17, U18, U19, U20, U21, U22, U23, U24, U25, U26, U27, U28: ~, Proj_footprint:SIZ200DT, symbol SIZ200DT:SIZ200
Connections:
- net +5V: now also J1.5 (Pin_5); no longer J1.1 (Pin_1)
- net ALARM: now also U15.2 (PC13); no longer U15.56 (PB4)
- net ESC1_VS1: now also U17.3 (S1/D2)
- net ESC1_VS2: now also U18.3 (S1/D2)
- net ESC1_VS3: now also U19.3 (S1/D2)
- net ESC2_VS1: now also U20.3 (S1/D2)
- net ESC2_VS2: now also U21.3 (S1/D2)
- net ESC2_VS3: now also U22.3 (S1/D2)
- net ESC3_VS1: now also U26.3 (S1/D2)
- net ESC3_VS2: now also U27.3 (S1/D2)
- net ESC3_VS3: now also U28.3 (S1/D2)
- net ESC4_VS1: now also U23.3 (S1/D2)
- net ESC4_VS2: now also U24.3 (S1/D2)
- net ESC4_VS3: now also U25.3 (S1/D2)
- net GND: now also U17.4 (S2), U18.4 (S2), U19.4 (S2), U20.4 (S2), U21.4 (S2), U22.4 (S2), U23.4 (S2), U24.4 (S2), U25.4 (S2), U26.4 (S2), U27.4 (S2), U28.4 (S2)
- net SPI2_CLK: now also J1.2 (Pin_2); no longer J1.5 (Pin_5)
- net SPI2_CS: now also J1.1 (Pin_1); no longer J1.2 (Pin_2)
- net SPI2_MISO: now also J1.3 (Pin_3); no longer J1.4 (Pin_4)
- net SPI2_MOSI: now also J1.4 (Pin_4); no longer J1.3 (Pin_3)
- net V_BAT: now also U17.2 (D1), U18.2 (D1), U19.2 (D1), U20.2 (D1), U21.2 (D1), U22.2 (D1), U23.2 (D1), U24.2 (D1), U25.2 (D1), U26.2 (D1), U27.2 (D1), U28.2 (D1)
- net at R46.2: now also U23.1 (G1)
- net at R67.2: now also U22.5 (G2)
- net at R5.2: now also U17.5 (G2)
- net at R4.2: now also U17.1 (G1)
- net at R66.2: now also U22.1 (G1)
- net at R69.2: now also U25.5 (G2)
- net at R68.2: now also U25.1 (G1)
- net at R32.2: now also U28.5 (G2)
- net at R17.2: now also U18.1 (G1)
- net at R57.2: now also U21.5 (G2)
- net at R56.2: now also U21.1 (G1)
- net at R43.2: now also U20.1 (G1)
- net at R44.2: now also U20.5 (G2)
- net at R47.2: now also U23.5 (G2)
- net at R20.2: now also U27.5 (G2)
- net at R8.2: now also U26.5 (G2)
- net at R30.2: now also U19.5 (G2)
- net at R59.2: now also U24.5 (G2)
- net at R29.2: now also U19.1 (G1)
- net at R18.2: now also U18.5 (G2)
- net at R19.2: now also U27.1 (G1)
- net at R7.2: now also U26.1 (G1)
- net at R31.2: now also U28.1 (G1)
- net at R58.2: now also U24.1 (G1)
- net BOOT1: no longer names the net of U15.28 (PB2)

Commit message: update routing
Connections:
- net 3V3_DEBUGGER: now also J2.3 (Pin_3); no longer J2.1 (Pin_1)
- net LED_BLUE: now also U15.59 (PB7); no longer U15.57 (PB5)
- net at U16.5 (VOUT): now also J2.1 (Pin_1); no longer J2.3 (Pin_3)
Other:
- moved on the sheet: C2, J2
Changed lines of the file:
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@@
   (junction (at 180.34 264.16) (diameter 0) (color 0 0 0 0)
   )
-  (junction (at 283.21 375.92) (diameter 0) (color 0 0 0 0)
+  (junction (at 283.21 378.46) (diameter 0) (color 0 0 0 0)
   )
   (junction (at 180.34 115.57) (diameter 0) (color 0 0 0 0)
@@
   (junction (at 388.62 256.54) (diameter 0) (color 0 0 0 0)
   )
-  (junction (at 283.21 373.38) (diameter 0) (color 0 0 0 0)
+  (junction (at 283.21 375.92) (diameter 0) (color 0 0 0 0)
   )
   (junction (at 62.23 115.57) (diameter 0) (color 0 0 0 0)
@@
   (junction (at 98.425 177.165) (diameter 0) (color 0 0 0 0)
   )
-  (junction (at 283.21 370.84) (diameter 0) (color 0 0 0 0)
+  (junction (at 283.21 373.38) (diameter 0) (color 0 0 0 0)
   )
   (junction (at 325.12 115.57) (diameter 0) (color 0 0 0 0)
@@
     (stroke (width 0) (type default))
   )
-  (wire (pts (xy 283.21 368.3) (xy 283.21 370.84))
+  (wire (pts (xy 283.21 370.84) (xy 283.21 373.38))
     (stroke (width 0) (type default))
   )
@@
     (stroke (width 0) (type default))
   )
-  (wire (pts (xy 283.21 373.38) (xy 283.21 375.92))
+  (wire (pts (xy 283.21 375.92) (xy 283.21 378.46))
     (stroke (width 0) (type default))
   )
@@
     (stroke (width 0) (type default))
   )
-  (wire (pts (xy 245.11 370.84) (xy 270.51 370.84))
-    (stroke (width 0) (type default))
-  )
   (wire (pts (xy 53.34 262.89) (xy 53.34 264.16))
     (stroke (width 0) (type default))
@@
     (stroke (width 0) (type default))
   )
-  (wire (pts (xy 283.21 375.92) (xy 283.21 377.825))
+  (wire (pts (xy 283.21 378.46) (xy 283.21 380.365))
     (stroke (width 0) (type default))
   )
@@
     (stroke (width 0) (type default))
   )
-  (wire (pts (xy 270.51 368.3) (xy 267.335 368.3))
+  (wire (pts (xy 245.11 370.84) (xy 270.51 370.84))
     (stroke (width 0) (type default))
   )
@@
     (stroke (width 0) (type default))
   )
-  (wire (pts (xy 283.21 370.84) (xy 283.21 373.38))
+  (wire (pts (xy 283.21 373.38) (xy 283.21 375.92))
     (stroke (width 0) (type default))
   )
@@
     )
   )
-  (global_label "LED_BLUE" (shape input) (at 554.355 97.79 0) (fields_autoplaced)
+  (global_label "LED_BLUE" (shape input) (at 554.355 102.87 0) (fields_autoplaced)
     (effects (font (size 1.27 1.27)) (justify left))
-    (property "Intersheetrefs" "${INTERSHEET_REFS}" (at 566.5325 97.79 0)
+    (property "Intersheetrefs" "${INTERSHEET_REFS}" (at 566.5325 102.87 0)
       (effects (font (size 1.27 1.27)) (justify left) hide)
     )
@@
     )
   )
-  (global_label "3V3_ESC" (shape input) (at 270.51 375.92 180) (fields_autoplaced)
+  (global_label "3V3_ESC" (shape input) (at 270.51 378.46 180) (fields_autoplaced)
     (effects (font (size 1.27 1.27)) (justify right))
-    (property "Intersheetrefs" "${INTERSHEET_REFS}" (at 259.4211 375.92 0)
+    (property "Intersheetrefs" "${INTERSHEET_REFS}" (at 259.4211 378.46 0)
       (effects (font (size 1.27 1.27)) (justify right) hide)
     )
@@
     )
   )
-  (global_label "3V3_FC" (shape input) (at 270.51 373.38 180) (fields_autoplaced)
+  (global_label "3V3_FC" (shape input) (at 270.51 375.92 180) (fields_autoplaced)
     (effects (font (size 1.27 1.27)) (justify right))
-    (property "Intersheetrefs" "${INTERSHEET_REFS}" (at 260.691 373.38 0)
+    (property "Intersheetrefs" "${INTERSHEET_REFS}" (at 260.691 375.92 0)
       (effects (font (size 1.27 1.27)) (justify right) hide)
     )
@@
     )
   )
-  (global_label "LED_PWR_3V3" (shape input) (at 283.21 368.3 0) (fields_autoplaced)
+  (global_label "LED_PWR_3V3" (shape input) (at 283.21 370.84 0) (fields_autoplaced)
     (effects (font (size 1.27 1.27)) (justify left))
-    (property "Intersheetrefs" "${INTERSHEET_REFS}" (at 299.0765 368.3 0)
+    (property "Intersheetrefs" "${INTERSHEET_REFS}" (at 299.0765 370.84 0)
       (effects (font (size 1.27 1.27)) (justify left) hide)
     )
@@
     )
   )
-  (global_label "3V3_DEBUGGER" (shape input) (at 267.335 368.3 180) (fields_autoplaced)
+  (global_label "3V3_DEBUGGER" (shape input) (at 270.51 373.38 180) (fields_autoplaced)
     (effects (font (size 1.27 1.27)) (justify right))
-    (property "Intersheetrefs" "${INTERSHEET_REFS}" (at 249.8961 368.3 0)
+    (property "Intersheetrefs" "${INTERSHEET_REFS}" (at 253.0711 373.38 0)
       (effects (font (size 1.27 1.27)) (justify right) hide)
     )
@@
     )
   )
-  (symbol (lib_id "Connector_Generic:Conn_02x04_Odd_Even") (at 275.59 370.84 0) (unit 1)
+  (symbol (lib_id "Connector_Generic:Conn_02x04_Odd_Even") (at 275.59 373.38 0) (unit 1)
     (in_bom yes) (on_board yes) (dnp no) (fields_autoplaced)
-    (property "Reference" "J2" (at 276.86 362.585 0)
+    (property "Reference" "J2" (at 276.86 365.125 0)
       (effects (font (size 1.27 1.27)))
     )
-    (property "Value" "Conn_02x04_Odd_Even" (at 276.86 365.125 0)
+    (property "Value" "Conn_02x04_Odd_Even" (at 276.86 367.665 0)
       (effects (font (size 1.27 1.27)))
     )
-    (property "Footprint" "Proj_footprint:PinHeader_2x04_P1.27mm_Vertical_SMD" (at 275.59 370.84 0)
+    (property "Footprint" "Proj_footprint:PinHeader_2x04_P1.27mm_Vertical_SMD" (at 275.59 373.38 0)
       (effects (font (size 1.27 1.27)) hide)
     )
-    (property "Datasheet" "~" (at 275.59 370.84 0)
+    (property "Datasheet" "~" (at 275.59 373.38 0)
       (effects (font (size 1.27 1.27)) hide)
     )
@@
     )
   )
-  (symbol (lib_id "Device:C_Small") (at 283.21 380.365 0) (unit 1)
+  (symbol (lib_id "Device:C_Small") (at 283.21 382.905 0) (unit 1)
     (in_bom yes) (on_board yes) (dnp no)
-    (property "Reference" "C2" (at 285.75 379.095 0)
+    (property "Reference" "C2" (at 285.75 381.635 0)
       (effects (font (size 1.27 1.27)) (justify left))
     )
-    (property "Value" "100uF" (at 285.115 382.27 0)
+    (property "Value" "100uF" (at 285.115 384.81 0)
       (effects (font (size 1.27 1.27)) (justify left))
     )
-    (property "Footprint" "Capacitor_SMD:C_1210_3225Metric_Pad1.33x2.70mm_HandSolder" (at 283.21 380.365 0)
+    (property "Footprint" "Capacitor_SMD:C_1210_3225Metric_Pad1.33x2.70mm_HandSolder" (at 283.21 382.905 0)
       (effects (font (size 1.27 1.27)) hide)
     )
-    (property "Datasheet" "~" (at 283.21 380.365 0)
+    (property "Datasheet" "~" (at 283.21 382.905 0)
       (effects (font (size 1.27 1.27)) hide)
     )
@@
     )
   )
-  (symbol (lib_id "power:GND") (at 283.21 382.905 0) (unit 1)
+  (symbol (lib_id "power:GND") (at 283.21 385.445 0) (unit 1)
     (in_bom yes) (on_board yes) (dnp no) (fields_autoplaced)
-    (property "Reference" "#PWR03" (at 283.21 389.255 0)
+    (property "Reference" "#PWR03" (at 283.21 391.795 0)
       (effects (font (size 1.27 1.27)) hide)
     )
-    (property "Value" "GND" (at 283.21 387.35 0)
+    (property "Value" "GND" (at 283.21 389.89 0)
       (effects (font (size 1.27 1.27)))
     )
-    (property "Footprint" "" (at 283.21 382.905 0)
+    (property "Footprint" "" (at 283.21 385.445 0)
       (effects (font (size 1.27 1.27)) hide)
     )
-    (property "Datasheet" "" (at 283.21 382.905 0)
+    (property "Datasheet" "" (at 283.21 385.445 0)
       (effects (font (size 1.27 1.27)) hide)
     )

Commit message: update routing
Parts:
- removed J3: ST-LINK, Proj_footprint:MountingPad_1x4, symbol Connector_Generic:Conn_01x04
- removed U1, U2, U7, U8: EFM8BB21, Proj_footprint:QFN-20-1EP_3x3mm_P0.5mm_EP1.8x1.8mm, symbol EFM8BB21:EFM8BB21
- removed U10, U4, U5, U9: FD6288Q, Package_DFN_QFN:QFN-24-1EP_4x4mm_P0.5mm_EP2.7x2.6mm, symbol FD6288:FD6288Q
- removed U12: MPU-6000, Proj_footprint:QFN-24-1EP_4x4mm_P0.5mm_EP2.15x2.15mm, symbol EFM8BB21:MPU-6000
- removed U16: RT9013-33GB, Package_TO_SOT_SMD:SOT-23-5, symbol RT9013:RT9013-33GB
- added J5: ST-LINK, Proj_footprint:STLINK_Port, symbol Connector_Generic:Conn_01x05
- added U1, U2, U7, U8: ~, Proj_footprint:QFN-20-1EP_3x3mm_P0.5mm_EP1.8x1.8mm, symbol EFM8BB21F16:EFM8BB21F16
- added U10: ~, Proj_footprint:QFN-24-1EP_4x4mm_P0.5mm_EP2.15x2.15mm, symbol MPU6000:MPU6000
- added U12: RT9013-33GB, Proj_footprint:SOT65P210X110-6N, symbol RT9013:RT9013-33GB
- added U29, U4, U5, U9: ~, Proj_footprint:QFN-24-1EP_4x4mm_P0.5mm_EP2.15x2.15mm, symbol FD6288Q:FD6288Q
- U3: footprint Proj_footprint:PDSO-G8_EP2.95x4.9mm_Mask2.4x3.1mm -> Proj_footprint:SOIC-8-1EP_3.9x4.9mm_P1.27mm_EP2.29x3mm
Connections:
- net +5V: now also U12.1 (VIN), U29.4 (VCC), U4.4 (VCC), U5.4 (VCC), U9.4 (VCC)
- net 3V3_DEBUGGER: now also J5.1 (Pin_1)
- net 3V3_ESC: now also U1.4 (VDD), U2.4 (VDD), U7.4 (VDD), U8.4 (VDD)
- net 3V3_FC: now also U10.13 (VDD)
- net ESC1_Acom: now also U1.15 (P0.7), U29.1 (LIN1)
- net ESC1_Apwm: now also U1.16 (P0.6), U29.22 (HIN1)
- net ESC1_Bcom: now also U1.13 (P1.1), U29.2 (LIN2)
- net ESC1_Bpwm: now also U1.14 (P1.0), U29.23 (HIN2)
- net ESC1_C2CK: now also U1.5 (RSTb/C2CK)
- net ESC1_C2D: now also U1.6 (P2.0/C2D)
- net ESC1_COM: now also U1.20 (P0.2)
- net ESC1_Ccom: now also U1.10 (P1.3), U29.3 (LIN3)
- net ESC1_Cpwm: now also U1.11 (P1.2), U29.24 (HIN3)
- net ESC1_HO1: now also U29.19 (HO1)
- net ESC1_HO2: now also U29.16 (HO2)
- net ESC1_HO3: now also U29.13 (HO3)
- net ESC1_LO1: now also U29.11 (LO1)
- net ESC1_LO2: now also U29.10 (LO2)
- net ESC1_LO3: now also U29.9 (LO3)
- net ESC1_MA: now also U1.19 (P0.3)
- net ESC1_MB: now also U1.18 (P0.4)
- net ESC1_MC: now also U1.17 (P0.5)
- net ESC1_RX: now also U1.2 (P0.0)
- net ESC1_VB1: now also U29.20 (VB1)
- net ESC1_VB2: now also U29.17 (VB2)
- net ESC1_VB3: now also U29.14 (VB3)
- net ESC1_VS1: now also U29.18 (VS1)
- net ESC1_VS2: now also U29.15 (VS2)
- net ESC1_VS3: now also U29.12 (VS3)
- net ESC2_Acom: now also U2.15 (P0.7), U4.1 (LIN1)
- net ESC2_Apwm: now also U2.16 (P0.6), U4.22 (HIN1)
- net ESC2_Bcom: now also U2.13 (P1.1), U4.2 (LIN2)
- net ESC2_Bpwm: now also U2.14 (P1.0), U4.23 (HIN2)
- net ESC2_C2CK: now also U2.5 (RSTb/C2CK)
- net ESC2_C2D: now also U2.6 (P2.0/C2D)
- net ESC2_COM: now also U2.20 (P0.2)
- net ESC2_Ccom: now also U2.10 (P1.3), U4.3 (LIN3)
- net ESC2_Cpwm: now also U2.11 (P1.2), U4.24 (HIN3)
- net ESC2_HO1: now also U4.19 (HO1)
- net ESC2_HO2: now also U4.16 (HO2)
- net ESC2_HO3: now also U4.13 (HO3)
- net ESC2_LO1: now also U4.11 (LO1)
- net ESC2_LO2: now also U4.10 (LO2)
- net ESC2_LO3: now also U4.9 (LO3)
- net ESC2_MA: now also U2.19 (P0.3)
- net ESC2_MB: now also U2.18 (P0.4)
- net ESC2_MC: now also U2.17 (P0.5)
- net ESC2_RX: now also U2.2 (P0.0)
- net ESC2_VB1: now also U4.20 (VB1)
- net ESC2_VB2: now also U4.17 (VB2)
- net ESC2_VB3: now also U4.14 (VB3)
- net ESC2_VS1: now also U4.18 (VS1)
- net ESC2_VS2: now also U4.15 (VS2)
- net ESC2_VS3: now also U4.12 (VS3)
- net ESC3_Acom: now also U7.15 (P0.7), U9.1 (LIN1)
- net ESC3_Apwm: now also U7.16 (P0.6), U9.22 (HIN1)
- net ESC3_Bcom: now also U7.13 (P1.1), U9.2 (LIN2)
- net ESC3_Bpwm: now also U7.14 (P1.0), U9.23 (HIN2)
- net ESC3_C2CK: now also U7.5 (RSTb/C2CK)
- net ESC3_C2D: now also U7.6 (P2.0/C2D)
- net ESC3_COM: now also U7.20 (P0.2)
- net ESC3_Ccom: now also U7.10 (P1.3), U9.3 (LIN3)
- net ESC3_Cpwm: now also U7.11 (P1.2), U9.24 (HIN3)
- net ESC3_HO1: now also U9.19 (HO1)
- net ESC3_HO2: now also U9.16 (HO2)
- net ESC3_HO3: now also U9.13 (HO3)
- net ESC3_LO1: now also U9.11 (LO1)
- net ESC3_LO2: now also U9.10 (LO2)
- net ESC3_LO3: now also U9.9 (LO3)
- net ESC3_MA: now also U7.19 (P0.3)
- net ESC3_MB: now also U7.18 (P0.4)
- net ESC3_MC: now also U7.17 (P0.5)
- net ESC3_RX: now also U7.2 (P0.0)
- net ESC3_VB1: now also U9.20 (VB1)
- net ESC3_VB2: now also U9.17 (VB2)
- net ESC3_VB3: now also U9.14 (VB3)
- net ESC3_VS1: now also U9.18 (VS1)
- net ESC3_VS2: now also U9.15 (VS2)
- net ESC3_VS3: now also U9.12 (VS3)
- net ESC4_Acom: now also U5.1 (LIN1), U8.15 (P0.7)
- net ESC4_Apwm: now also U5.22 (HIN1), U8.16 (P0.6)
- net ESC4_Bcom: now also U5.2 (LIN2), U8.13 (P1.1)
- net ESC4_Bpwm: now also U5.23 (HIN2), U8.14 (P1.0)
- net ESC4_C2CK: now also U8.5 (RSTb/C2CK)
- net ESC4_C2D: now also U8.6 (P2.0/C2D)
- net ESC4_COM: now also U8.20 (P0.2)
- net ESC4_Ccom: now also U5.3 (LIN3), U8.10 (P1.3)
- net ESC4_Cpwm: now also U5.24 (HIN3), U8.11 (P1.2)
- net ESC4_HO1: now also U5.19 (HO1)
- net ESC4_HO2: now also U5.16 (HO2)
- net ESC4_HO3: now also U5.13 (HO3)
- net ESC4_LO1: now also U5.11 (LO1)
- net ESC4_LO2: now also U5.10 (LO2)
- net ESC4_LO3: now also U5.9 (LO3)
- net ESC4_MA: now also U8.19 (P0.3)
- net ESC4_MB: now also U8.18 (P0.4)
- net ESC4_MC: now also U8.17 (P0.5)
- net ESC4_RX: now also U8.2 (P0.0)
- net ESC4_VB1: now also U5.20 (VB1)
- net ESC4_VB2: now also U5.17 (VB2)
- net ESC4_VB3: now also U5.14 (VB3)
- net ESC4_VS1: now also U5.18 (VS1)
- net ESC4_VS2: now also U5.15 (VS2)
- net ESC4_VS3: now also U5.12 (VS3)
- net GND: now also U6.29 (GND), J5.5 (Pin_5), U1.12 (GND), U1.21 (GND), U1.3 (GND), U10.1 (CLKIN), U10.11 (FSYNC), U10.18 (GND), U10.25 (GND), U12.2 (GND), U2.12 (GND), U2.21 (GND), U2.3 (GND), U29.25 (GND), U29.6 (COM), U4.25 (GND), U4.6 (COM), U5.25 (GND), U5.6 (COM), U7.12 (GND), U7.21 (GND), U7.3 (GND), U8.12 (GND), U8.21 (GND), U8.3 (GND), U9.25 (GND), U9.6 (COM)
- net IMU_CLK: now also U10.23 (SCL/SCLK)
- net IMU_CS: now also U10.8 (nCS)
- net IMU_INT: now also U10.12 (INT)
- net IMU_MISO: now also U10.9 (SDO/AD0)
- net IMU_MOSI: now also U10.24 (SDA/SD1)
- net STM32_CLK: now also J5.3 (Pin_3)
- net STM32_DIO: now also J5.2 (Pin_2)
- net at C34.1: now also U10.20 (CPOUT)
- net at J2.1 (Pin_1): now also U12.5 (VOUT)
- net STM32_NRST: now reaches R83.2, U15.7 (NRST)
- net STM32_NRST: now also J5.4 (Pin_4)
- net at C33.1: now also U10.10 (REGOUT)
