File: FC_ESC_STM32F405RG_26x26.kicad_pcb (KiCad board)
At the start: 8 copper layers, 34 x 34 mm, 211 parts, among them J1 SPI, J12 Conn_02x02_Odd_Even, J14 UART1, J15 UART3_I2C2, J16 MOTOR, J17 MOTOR, J18 MOTOR, J19 MOTOR, J2 Conn_02x04_Odd_Even, J20 USB_A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

Commit message: add dimension
Routing:
- net 3V3_FC: track 136.8 -> 136.9 mm, vias 29 -> 30
- net V_BAT: track 4.92 -> 4.90 mm, vias 74 -> 75
